Commit message: 2nd git commit, robot is working, gui isn't popping up

File: urdf/robot.urdf (robot description, URDF)
Before this commit: robot macs_robot, 6 links, 5 joints
Links:
- link laser_horiz: geometry collision cylinder length=0.072 radius=0.052; visual cylinder length=0.072 radius=0.052
- link laser_vert_bottom: geometry collision box size=0.062 0.062 0.087; visual box size=0.062 0.062 0.087
- link laser_vert_top_left: geometry collision box size=0.062 0.062 0.087; visual box size=0.062 0.062 0.087
- link laser_vert_top_right: geometry collision box size=0.062 0.062 0.087; visual box size=0.062 0.062 0.087

File: urdf/robot.xacro (robot description, xacro)
@@ -1,7 +1,11 @@
 <?xml version="1.0"?>
 <robot xmlns:xacro="http://www.ros.org/wiki/xacro" name="macs_robot">
+    <!-- Include the XACRO file that defines a Hokuyo LIDAR. -->
+<xacro:include filename="$(find gazebo_plugins)/test/multi_robot_scenario/xacro/laser/hokuyo.xacro" />
+    <!-- Include the XACRO file that defines a Hokuyo LIDAR. -->
+<xacro:include filename="$(find velodyne_description)/urdf/VLP-16.urdf.xacro"/>
   <link name="base">
     <visual>
-      <origin xyz="0 0 0" rpy="0 0 0"/>
+      <origin xyz="-0.2 0 .93" rpy="0 0 0"/>
       <geometry>
         <box size="0.94 0.78 1.98"/>
@@ -12,5 +16,5 @@
     </visual>
     <collision>
-      <origin xyz="0 0 0" rpy="0 0 0"/>
+      <origin xyz="-0.2 0 .93" rpy="0 0 0"/>
       <geometry>
         <box size="0.94 0.78 1.98"/>
@@ -18,74 +22,12 @@
     </collision>
   </link>
-    <link name="laser_vert_bottom">
-    <visual>
-      <origin xyz="0 0 0" rpy="0 0 0"/>
-      <geometry>
-        <box size="0.62 0.62 0.87"/>
-      </geometry>
-      <material name="Cyan">
-      	<color rgba="0 1.0 1.0 1.0"/>
-      </material>
-    </visual>
-    <collision>
-      <origin xyz="0 0 0" rpy="0 0 0"/>
-      <geometry>
-        <box size="0.62 0.62 0.87"/>
-      </geometry>
-    </collision>
-  </link>
-  <link name="laser_vert_top_right">
-    <visual>
-      <origin xyz="0 0 0" rpy="0 0 0"/>
-      <geometry>
-        <box size="0.62 0.62 0.87"/>
-      </geometry>
-      <material name="Cyan">
-      	<color rgba="0 1.0 1.0 1.0"/>
-      </material>
-    </visual>
-    <collision>
-      <origin xyz="0 0 0" rpy="0 0 0"/>
-      <geometry>
-        <box size="0.62 0.62 0.87"/>
-      </geometry>
-    </collision>
-  </link>
-  <link name="laser_vert_top_left">
-    <visual>
-      <origin xyz="0 0 0" rpy="0 0 0"/>
-      <geometry>
-        <box size="0.62 0.62 0.87"/>
-      </geometry>
-      <material name="Cyan">
-      	<color rgba="0 1.0 1.0 1.0"/>
-      </material>
-    </visual>
-    <collision>
-      <origin xyz="0 0 0" rpy="0 0 0"/>
-      <geometry>
-        <box size="0.62 0.62 0.87"/>
-      </geometry>
-    </collision>
-  </link>
-  <link name="laser_horiz">
-    <visual>
-      <origin xyz="0 0 0" rpy="0 0 0"/>
-      <geometry>
-        <cylinder radius="0.52" length="0.72"/>
-      </geometry>
-      <material name="Cyan">
-      	<color rgba="0 1.0 1.0 1.0"/>
-      </material>
-    </visual>
-    <collision>
-      <origin xyz="0 0 0" rpy="0 0 0"/>
-      <geometry>
-        <cylinder radius="0.52" length="0.72"/>
-      </geometry>
-    </collision>
-  </link>
+    <xacro:laser name="laser_vert_bottom" parent="base" xyz="0.3157894464801903 -0.002068548615034871 0.5099999434059285" rpy="3.1354753 -1.3045001 0.0024658" meshes="package://gazebo_plugins/test/multi_robot_scenario/meshes/laser" />
+    <xacro:laser name="laser_vert_top_right" parent="base" xyz="0.2978 -0.1450 1.8451" rpy="-1.1760 0.6313 1.9377" meshes="package://gazebo_plugins/test/multi_robot_scenario/meshes/laser" />
+    <xacro:laser name="laser_vert_top_left" parent="base" xyz="0.2997 0.1531 1.8451" rpy="1.1760 0.6198 1.9560" meshes="package://gazebo_plugins/test/multi_robot_scenario/meshes/laser" />
+  <!-- Invoke the macro to define the Hokuyo LIDAR. -->
+  <VLP-16 parent="base" name="laser_horiz" topic="laser_horiz/packets" hz="10" samples="440" gpu="false">
+    <origin xyz="0.2325416305773505 -0.0001380069427607134 1.920122926231907" rpy="-0.0012068 0.114646 -0.0015308" />
+  </VLP-16>
   <xacro:macro name="xacro_name" params="suffix reflect">
-   <!-- <xacro:xacro_name suffix="left" reflect="1" /> -->
     <link name="wheel__${suffix}">
     <visual>
@@ -108,30 +50,26 @@
   <xacro:xacro_name suffix="left" reflect="1" />
   <xacro:xacro_name suffix="right" reflect="-1" />
-  <joint name="base_laser_vert_bottom_joint" type="fixed">
-    <parent link="base"/>
-    <child link="laser_vert_bottom"/>
-    <origin xyz="0.3158 -0.0021 0.5100" rpy="3.1355 -1.3045 0.0025"/>
-  </joint>
-  <joint name="base_laser_vert_top_right_joint" type="fixed">
-    <parent link="base"/>
-    <child link="laser_vert_top_right"/>
-    <origin xyz="0.2978 -0.1450 1.8451" rpy="-1.1760 0.6313 -1.9377"/>
-  </joint>
-  <joint name="base_laser_vert_top_left_joint" type="fixed">
-    <parent link="base"/>
-    <child link="laser_vert_top_left"/>
-    <origin xyz="0.2997 0.1531 1.8443" rpy="1.1780 0.6198 1.9560"/>
-  </joint>
-  <joint name="base_laser_horiz_joint" type="fixed">
-    <parent link="base"/>
-    <child link="laser_horiz"/>
-    <origin xyz="0.2325 0.0001 1.9201" rpy="-0.0012 0.1146 -0.0015"/>
-  </joint>
+      <link name="wheel__center">
+    <visual>
+      <origin xyz="0 0 0" rpy="0 0 0"/>
+      <geometry>
+        <cylinder radius="0.15" length="0.05"/>
+      </geometry>
+      <material name="Cyan">
+      	<color rgba="0 1.0 1.0 1.0"/>
+      </material>
+    </visual>
+    <collision>
+      <origin xyz="0 0 0" rpy="0 0 0"/>
+      <geometry>
+        <cylinder radius="0.15" length="0.05"/>
+      </geometry>
+    </collision>
+  </link>
   <xacro:macro name="xacro_name" params="suffix reflect">
-   <!-- <xacro:xacro_name suffix="left" reflect="1" /> -->
-  <joint name="base_wheel__${suffix}_joint" type="fixed">
+  <joint name="base_wheel__${suffix}_joint" type="continuous">
     <parent link="base"/>
     <child link="wheel__${suffix}"/>
-    <origin xyz="-0.10 0.4 0.0" rpy="${-pi/2} 0.0 0.0"/>
+    <origin xyz="-0.10 ${reflect * 0.4} 0.0" rpy="${-pi/2} 0.0 0.0"/>
     <limit effort="1.0" velocity="1.0"/>
   </joint>
@@ -139,3 +77,9 @@
   <xacro:xacro_name suffix="left" reflect="1" />
   <xacro:xacro_name suffix="right" reflect="-1" />
+  <joint name="base_wheel__center_joint" type="continuous">
+    <parent link="base"/>
+    <child link="wheel__center"/>
+    <origin xyz="0.10 0.0 0.0" rpy="${-pi/2} 0.0 0.0"/>
+    <limit effort="1.0" velocity="1.0"/>
+  </joint>
 </robot>

Commit message: Robot launches along with joint state publisher and GUI if desired

File: urdf/robot.urdf (robot description, URDF)
Before this commit: robot macs_robot, 6 links, 5 joints
Links:
- added link wheel_center; collision cylinder length=0.05 radius=0.15; visual cylinder length=0.05 radius=0.15
- added link wheel_right; collision cylinder length=0.05 radius=0.2; visual cylinder length=0.05 radius=0.2
Joints:
- added joint base_wheel_center_joint: type continuous, parent base, child wheel_center, origin xyz=-0.10 0.0 0.0 rpy=-1.57 0.0 0.0, limit effort=1.0 velocity=1.0
- added joint base_wheel_right_joint: type continuous, parent base, child wheel_right, origin xyz=-0.10 -0.4 0.0 rpy=-1.57 0.0 0.0, limit effort=1.0 velocity=1.0
- joint base_wheel_left_joint: type fixed -> continuous

Commit message: Altered robot base origin to half height. Removed publishing line from launch file.

File: urdf/robot.urdf (robot description, URDF)
Before this commit: robot macs_robot, 8 links, 7 joints
Joints:
- joint base_wheel_center_joint: origin xyz=-0.10 0.0 0.0 rpy=-1.57 0.0 0.0 -> xyz=0.10 0.0 0.0 rpy=-1.57 0.0 0.0

File: urdf/robot.xacro (robot description, xacro)
@@ -7,5 +7,5 @@
   <link name="base">
     <visual>
-      <origin xyz="-0.2 0 .93" rpy="0 0 0"/>
+      <origin xyz="-0.2 0 .99" rpy="0 0 0"/>
       <geometry>
         <box size="0.94 0.78 1.98"/>
@@ -16,5 +16,5 @@
     </visual>
     <collision>
-      <origin xyz="-0.2 0 .93" rpy="0 0 0"/>
+      <origin xyz="-0.2 0 .99" rpy="0 0 0"/>
       <geometry>
         <box size="0.94 0.78 1.98"/>
