Commit message: third commit

File: urdf/urdf_from_xacro.urdf (robot description, URDF)
Before this commit: robot macs_robot, 5 links, 4 joints
Links:
- added link base_link
- added link imu; collision sphere radius=0.1; visual sphere radius=0.1
- added link laser_horiz_base_link, mass 0.83; collision cylinder length=0.0717 radius=0.0516; visual mesh filename=package://velodyne_description/meshes/VLP16_base_1.dae
- added link wheel__center; collision cylinder length=0.05 radius=0.15; visual cylinder length=0.05 radius=0.15
- added link wheel__left; collision cylinder length=0.05 radius=0.2; visual cylinder length=0.05 radius=0.2
- added link wheel__right; collision cylinder length=0.05 radius=0.2; visual cylinder length=0.05 radius=0.2
- link laser_horiz: mass None -> 0.01; geometry visual mesh filename=package://velodyne_description/meshes/VLP16_scan.dae
- link laser_vert_bottom: mass None -> 1e-5; geometry collision box size=0.1 0.1 0.1; visual mesh filename=package://gazebo_plugins/test/multi_robot_scenario/meshes/l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
- link laser_vert_top_left: mass None -> 1e-5; geometry collision box size=0.1 0.1 0.1; visual mesh filename=package://gazebo_plugins/test/multi_robot_scenario/meshes/l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
- link laser_vert_top_right: mass None -> 1e-5; geometry collision box size=0.1 0.1 0.1; visual mesh filename=package://gazebo_plugins/test/multi_robot_scenario/meshes/l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
Joints:
- removed joint base_laser_horiz_joint
- added joint base_link_base_joint: type fixed, parent base_link, child base, origin xyz=0.07 0 1.792 rpy=0.0 3.14159265359 0.0
- added joint base_link_imu_joint: type fixed, parent base_link, child imu, origin xyz=0.0 0.0 0.0 rpy=3.1405788 0.0034281 3.1382064
- added joint base_wheel__center_joint: type continuous, parent base, child wheel__center, origin xyz=0.10 0.0 0.0 rpy=-1.57079632679 0.0 0.0, limit effort=1.0 velocity=1.0
- added joint base_wheel__left_joint: type continuous, parent base, child wheel__left, origin xyz=-0.10 0.4 0.0 rpy=-1.57079632679 0.0 0.0, limit effort=1.0 velocity=1.0
- added joint base_wheel__right_joint: type continuous, parent base, child wheel__right, origin xyz=-0.10 -0.4 0.0 rpy=-1.57079632679 0.0 0.0, limit effort=1.0 velocity=1.0
- added joint laser_horiz_base_mount_joint: type fixed, parent base, child laser_horiz_base_link, origin xyz=0.2325416305773505 -0.0001380069427607134 1.920122926231907 rpy=-0.0012068 0.114646 -0.0015308
- added joint laser_horiz_base_scan_joint: type fixed, parent laser_horiz_base_link, child laser_horiz, origin xyz=0 0 0.0377 rpy=0 0 0
- joint base_laser_vert_bottom_joint: axis (none) -> 0 0 1; origin xyz=0.3158 -0.0021 0.5100 rpy=3.1355 -1.3045 0.0025 -> xyz=0.3157894464801903 -0.002068548615034871 0.5099999434059285 rpy=3.1354753 -1.3045001 0.0024658
- joint base_laser_vert_top_left_joint: axis (none) -> 0 0 1; origin xyz=0.2997 0.1531 1.8443 rpy=1.1780 0.6198 1.9560 -> xyz=0.2997 0.1531 1.8451 rpy=1.1760 0.6198 1.9560
- joint base_laser_vert_top_right_joint: axis (none) -> 0 0 1; origin xyz=0.2978 -0.1450 1.8451 rpy=-1.1760 0.6313 -1.9377 -> xyz=0.2978 -0.1450 1.8451 rpy=-1.1760 0.6313 1.9377
